File: Project Documents/System Sketch.sch (EAGLE design)
At the start: 0 parts

Commit message: Updated System Sketch
Other:
- note added: "IR1"
- note added: "IR2"
- note added: "Motor Controller"
- note removed: "10"
- note removed: "11"
- note removed: "12"
- note removed: "9"
- note removed: "IR1 & 2"
- note removed: "IR3 & 4"
- note removed: "IR5"
- note removed: "Light Sensor"
- note removed: "Limit Switch"
- note removed: "Motor Driver"
- note removed: "Temperature"
