File: Project Documents/Schematic.sch (EAGLE design)
At the start: 13 parts, among them IC1 L298, IC2 L298

Commit message: Updated Robot Schematic for remapped pins
Parts:
- removed PH1: D1160_12, photo-elements:D1160_12
- removed R2A2: 10K, rcl:R-US_0309/12
Other:
- note removed: "Light Sensor"

Commit message: Updated the Schematic with removed components
Requirements of the project changed causing some components to be removed, IR3 -5, LS 1 and 2 and the addition of the potentiometer.
Other:
- note added: "Potentiometer"
- note removed: "IR3"
- note removed: "IR4"
- note removed: "IR5"
- note removed: "LS1"
- note removed: "LS2"
- moved on the sheet: DIS1, LED1, LED2, LED3, LED4, R2A, R2B, R2C, R2D

Commit message: Update Schematic.sch
Other:
- note added: "LS1"
- note added: "LS2"
- note removed: "HC-SR04"
- note removed: "Ultrasonic_Echo"
- note removed: "Ultrasonic_Trig"
Changed lines of the file:
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@@
 <text x="111.76" y="60.96" size="1.778" layer="93">M4-</text>
 <text x="20.32" y="20.32" size="1.778" layer="93">IR1</text>
-<text x="20.32" y="22.86" size="1.778" layer="93">IR2</text>
+<text x="-27.94" y="33.02" size="1.778" layer="93">IR2</text>
 <wire x1="-91.44" y1="17.78" x2="-83.82" y2="17.78" width="0.1524" layer="93"/>
 <wire x1="-91.44" y1="10.16" x2="-83.82" y2="10.16" width="0.1524" layer="93"/>
@@
 <text x="-86.36" y="-10.16" size="1.778" layer="93">5V</text>
 <text x="-86.36" y="-25.4" size="1.778" layer="93">GND</text>
-<text x="-86.36" y="-17.78" size="1.778" layer="93">PC9</text>
+<text x="-86.36" y="-17.78" size="1.778" layer="93">PA5</text>
 <wire x1="-91.44" y1="86.36" x2="-83.82" y2="86.36" width="0.1524" layer="93"/>
 <wire x1="-91.44" y1="73.66" x2="-83.82" y2="73.66" width="0.1524" layer="93"/>
@@
 <text x="-86.36" y="86.36" size="1.778" layer="93">5V</text>
 <text x="-86.36" y="73.66" size="1.778" layer="93">GND</text>
-<wire x1="-91.44" y1="114.3" x2="-83.82" y2="114.3" width="0.1524" layer="93"/>
-<wire x1="-91.44" y1="109.22" x2="-83.82" y2="109.22" width="0.1524" layer="93"/>
-<wire x1="-91.44" y1="104.14" x2="-83.82" y2="104.14" width="0.1524" layer="93"/>
-<wire x1="-91.44" y1="99.06" x2="-83.82" y2="99.06" width="0.1524" layer="93"/>
-<text x="-86.36" y="114.3" size="1.778" layer="93">5V</text>
-<text x="-86.36" y="99.06" size="1.778" layer="93">GND</text>
-<text x="-127" y="116.84" size="1.778" layer="93">HC-SR04</text>
-<text x="-40.64" y="43.18" size="1.778" layer="93">Ultrasonic_Trig</text>
-<text x="-40.64" y="38.1" size="1.778" layer="93">Ultrasonic_Echo</text>
 <text x="20.32" y="53.34" size="1.778" layer="93" ratio="5">T1</text>
 <text x="66.04" y="104.14" size="1.778" layer="93" ratio="5">PB3</text>
@@
 <text x="-96.52" y="30.48" size="1.778" layer="97" ratio="5">5V</text>
 <text x="-96.52" y="27.94" size="1.778" layer="97" ratio="5">GND</text>
-<text x="-86.36" y="104.14" size="1.778" layer="91">PA3</text>
-<text x="-86.36" y="109.22" size="1.778" layer="91">PA1</text>
 <text x="-86.36" y="81.28" size="1.778" layer="91">PA8</text>
 <text x="-40.64" y="40.64" size="1.778" layer="91">Potentiometer</text>
+<text x="-27.94" y="38.1" size="1.778" layer="91">LS1</text>
+<text x="-27.94" y="35.56" size="1.778" layer="91">LS2</text>
+<text x="58.42" y="-7.62" size="1.778" layer="91">GND</text>
+<text x="58.42" y="-30.48" size="1.778" layer="91">GND</text>
+<text x="58.42" y="7.62" size="1.778" layer="91">PA3</text>
+<text x="58.42" y="-15.24" size="1.778" layer="91">PA4</text>
 </plain>
 <moduleinsts>
@@
 <attribute name="NAME" x="-111.76" y="81.28" size="2.032" layer="95" align="bottom-center"/>
 </moduleinst>
-<moduleinst name="UTLRASONIC1" module="UTLRASONIC" x="-111.76" y="106.68">
-<attribute name="NAME" x="-111.76" y="106.68" size="2.032" layer="95" align="bottom-center"/>
+<moduleinst name="LIMITSWITCH1" module="LIMITSWITCH" x="88.9" y="0">
+<attribute name="NAME" x="88.9" y="0" size="2.032" layer="95" align="bottom-center"/>
+</moduleinst>
+<moduleinst name="LIMITSWITCH2" module="LIMITSWITCH" x="88.9" y="-22.86">
+<attribute name="NAME" x="88.9" y="-22.86" size="2.032" layer="95" align="bottom-center"/>
 </moduleinst>
 </moduleinsts>
@@
 </segment>
 </net>
+<net name="N$62" class="0">
+<segment>
+<portref moduleinst="LIMITSWITCH1" port="COM"/>
+<wire x1="68.58" y1="-7.62" x2="60.96" y2="-7.62" width="0.1524" layer="91"/>
+</segment>
+</net>
+<net name="N$63" class="0">
+<segment>
+<wire x1="60.96" y1="7.62" x2="68.58" y2="7.62" width="0.1524" layer="91"/>
+</segment>
+</net>
+<net name="N$64" class="0">
+<segment>
+<wire x1="60.96" y1="2.54" x2="68.58" y2="2.54" width="0.1524" layer="91"/>
+</segment>
+</net>
+<net name="N$65" class="0">
+<segment>
+<wire x1="60.96" y1="-15.24" x2="68.58" y2="-15.24" width="0.1524" layer="91"/>
+</segment>
+</net>
+<net name="N$66" class="0">
+<segment>
+<wire x1="60.96" y1="-20.32" x2="68.58" y2="-20.32" width="0.1524" layer="91"/>
+</segment>
+</net>
+<net name="N$67" class="0">
+<segment>
+<wire x1="60.96" y1="-30.48" x2="68.58" y2="-30.48" width="0.1524" layer="91"/>
+</segment>
+</net>
